Commit message: Updated

File: pet_bot_test5/urdf/pet_bot_test5.urdf.xacro (robot description, xacro)
@@ -8,16 +8,13 @@
     name="base_link">
     <inertial>
-      <origin
-        xyz="-0.00113291682806678 0.00312887171663282 -0.0086784545054986"
-        rpy="0 0 0" />
-      <mass
-        value="0.5" />
-      <inertia
-        ixx="0.000428558923538308"
-        ixy="2.71016532559896E-08"
-        ixz="-7.42171927160237E-08"
-        iyy="0.000104687926825432"
-        iyz="-1.98122646645251E-07"
-        izz="0.000444638895048129" />
+      <origin xyz="0 0 0" rpy="0 0 0"/>
+      <mass value="0.5"/>
+      <inertia
+        ixx="0.0004286"
+        iyy="0.0001047"
+        izz="0.0004446"
+        ixy="0"
+        ixz="0"
+        iyz="0"/>
     </inertial>
     <visual>

Commit message: Added Camera Sensor

File: pet_bot_test5/urdf/pet_bot_test5.urdf.xacro (robot description, xacro)
@@ -949,4 +949,29 @@
       effort="30.0"
       velocity="5.0" />
+  </joint>
+  <link name="camera_link">
+    <visual>
+      <geometry>
+        <box size="0.03 0.03 0.03"/>
+      </geometry>
+    </visual>
+    <collision>
+      <geometry>
+        <box size="0.03 0.03 0.03"/>
+      </geometry>
+    </collision>
+    <inertial>
+      <mass value="0.01"/>
+      <origin xyz="0 0 0"/>
+      <inertia
+        ixx="0.0001" ixy="0" ixz="0"
+        iyy="0.0001" iyz="0"
+        izz="0.0001"/>
+    </inertial>
+  </link>
+  <joint name="camera_joint" type="fixed">
+    <parent link="base_link"/>
+    <child link="camera_link"/>
+    <origin xyz="0.003 -0.13 0.030" rpy="0 0 -1.57"/>
   </joint>
   <!-- ROS 2 Control Hardware Interface for Ignition -->
@@ -1020,4 +1045,25 @@
     </joint>
   </ros2_control>
+  <!--camera link sensor-->
+  <gazebo reference="camera_link">
+    <sensor name="camera" type="camera">
+      <always_on>true</always_on>
+      <update_rate>30</update_rate>
+      <visualize>true</visualize>
+      <camera>
+        <horizontal_fov>1.047</horizontal_fov>
+        <image>
+          <width>640</width>
+          <height>480</height>
+          <format>R8G8B8</format>
+        </image>
+        <clip>
+          <near>0.1</near>
+          <far>100</far>
+        </clip>
+      </camera>
+      <topic>/camera</topic>
+    </sensor>
+  </gazebo>
   <!-- ================== TRANSMISSIONS FOR ALL 12 JOINTS ================== -->
   <!-- FRONT LEFT LEG -->
@@ -1170,3 +1216,10 @@
     </plugin>
   </gazebo-->
+  <gazebo>
+    <plugin
+        filename="ignition-gazebo-sensors-system"
+        name="ignition::gazebo::systems::Sensors">
+        <render_engine>ogre2</render_engine>
+    </plugin>
+  </gazebo>
 </robot>

Commit message: Added depth camera

File: pet_bot_test5/urdf/pet_bot_test5.urdf.xacro (robot description, xacro)
@@ -950,9 +950,12 @@
       velocity="5.0" />
   </joint>
-  <link name="camera_link">
+  <link name="depth_camera">
     <visual>
       <geometry>
         <box size="0.03 0.03 0.03"/>
       </geometry>
+      <material name="white">
+        <color rgba="1 1 1 1"/>
+      </material>
     </visual>
     <collision>
@@ -970,7 +973,7 @@
     </inertial>
   </link>
-  <joint name="camera_joint" type="fixed">
+  <joint name="depth_camera_joint" type="fixed">
     <parent link="base_link"/>
-    <child link="camera_link"/>
+    <child link="depth_camera"/>
     <origin xyz="0.003 -0.13 0.030" rpy="0 0 -1.57"/>
   </joint>
@@ -1046,8 +1049,8 @@
   </ros2_control>
   <!--camera link sensor-->
-  <gazebo reference="camera_link">
-    <sensor name="camera" type="camera">
+  <gazebo reference="depth_camera">
+    <sensor name="depth_camera" type="depth_camera">
       <always_on>true</always_on>
-      <update_rate>30</update_rate>
+      <update_rate>10</update_rate>
       <visualize>true</visualize>
       <camera>
@@ -1056,12 +1059,15 @@
           <width>640</width>
           <height>480</height>
-          <format>R8G8B8</format>
+          <!-- <format>R8G8B8</format> -->
         </image>
         <clip>
           <near>0.1</near>
-          <far>100</far>
+          <far>10.0</far>
         </clip>
       </camera>
-      <topic>/camera</topic>
+      <depth_camera>
+        <output>depth</output>
+      </depth_camera>
+      <topic>/depth_camera</topic>
     </sensor>
   </gazebo>
